File: 10m08sau324c8g_io_bnks.kicad_sch (KiCad schematic)
At the start: 14 parts

Commit message: Hierarchy to Flat completes
The hierarchy sheets have been converted into flat sheets and global labels have been used in appropriate place.
Parts:
- gave numbers to parts that had none: 6
