File: 10m08sau324c8g_io_dev.kicad_sch (KiCad schematic)
At the start: 82 parts

Commit message: Hierarchy to Flat completes
The hierarchy sheets have been converted into flat sheets and global labels have been used in appropriate place.
Parts:
- gave numbers to parts that had none: 82
Connections:
- net DIP_1: now also SW3.2; no longer SW3.1
- net GND: now also SW3.1; no longer SW3.2
Other:
- moved on the sheet: R14, R15, R16, R17, R18, SW3, SW4, SW5, SW6, SW7
