File: programmer.kicad_sch (KiCad schematic)
At the start: 27 parts

Commit message: Hierarchy to Flat completes
The hierarchy sheets have been converted into flat sheets and global labels have been used in appropriate place.
Parts:
- added J?: Conn_01x05, symbol Connector_Generic:Conn_01x05
- gave numbers to parts that had none: 27
Connections:
- net GND: now also J?.4 (Pin_4)
- new net FPGA_JTAG_TCK_HED: J?.2 (Pin_2)
- new net FPGA_JTAG_TDI_HED: J?.3 (Pin_3)
- new net FPGA_JTAG_TDO_HED: J?.5 (Pin_5)
- new net FPGA_JTAG_TMS_HED: J?.1 (Pin_1)
Other:
- moved on the sheet: C17

Commit message: Decoupling done
The decoupling for the 10CL025 was completed using the evaluation module as reference.
Parts:
- gave numbers to parts that had none: 1
Changed lines of the file:
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@@
 		(in_pos_files yes)
 		(dnp yes)
-		(property "Reference" "J?"
+		(property "Reference" "J4"
 			(at 242.57 126.238 0)
 			(show_name no)
@@
 			(project "STM32-FPGA"
 				(path "/ec7f004b-4356-4f5c-8bcf-777a271cc592"
-					(reference "J?")
+					(reference "J4")
 					(unit 1)
 				)
@@
 	(sheet_instances
 		(path "/"
-			(page "2")
-		)
-	)
+			(page "3")
+		)
+	)
