File: sdram.kicad_sch (KiCad schematic)
At the start: 11 parts

Commit message: Hierarchy to Flat completes
The hierarchy sheets have been converted into flat sheets and global labels have been used in appropriate place.
Parts:
- gave numbers to parts that had none: 11
Changed lines of the file:
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@@
 		(in_pos_files yes)
 		(dnp no)
-		(property "Reference" "C?"
+		(property "Reference" "C79"
 			(at 51.054 51.308 0)
 			(show_name no)
@@
 			(project "STM32-FPGA"
 				(path "/a5dcf55a-c00b-44e4-be21-50af8ba3dde4"
-					(reference "C?")
+					(reference "C79")
 					(unit 1)
 				)
@@
 		(in_pos_files yes)
 		(dnp no)
-		(property "Reference" "C?"
+		(property "Reference" "C82"
 			(at 77.724 51.308 0)
 			(show_name no)
@@
 			(project "STM32-FPGA"
 				(path "/a5dcf55a-c00b-44e4-be21-50af8ba3dde4"
-					(reference "C?")
+					(reference "C82")
 					(unit 1)
 				)
@@
 		(in_pos_files yes)
 		(dnp no)
-		(property "Reference" "C?"
+		(property "Reference" "C85"
 			(at 161.544 51.308 0)
 			(show_name no)
@@
 			(project "STM32-FPGA"
 				(path "/a5dcf55a-c00b-44e4-be21-50af8ba3dde4"
-					(reference "C?")
+					(reference "C85")
 					(unit 1)
 				)
@@
 		(dnp no)
 		(fields_autoplaced yes)
-		(property "Reference" "U?"
+		(property "Reference" "U4"
 			(at 92.202 50.038 0)
 			(show_name no)
@@
 			(project "STM32-FPGA"
 				(path "/a5dcf55a-c00b-44e4-be21-50af8ba3dde4"
-					(reference "U?")
+					(reference "U4")
 					(unit 1)
 				)
@@
 		(in_pos_files yes)
 		(dnp no)
-		(property "Reference" "C?"
+		(property "Reference" "C84"
 			(at 152.654 51.308 0)
 			(show_name no)
@@
 			(project "STM32-FPGA"
 				(path "/a5dcf55a-c00b-44e4-be21-50af8ba3dde4"
-					(reference "C?")
+					(reference "C84")
 					(unit 1)
 				)
@@
 		(in_pos_files yes)
 		(dnp no)
-		(property "Reference" "C?"
+		(property "Reference" "C81"
 			(at 68.834 51.308 0)
 			(show_name no)
@@
 			(project "STM32-FPGA"
 				(path "/a5dcf55a-c00b-44e4-be21-50af8ba3dde4"
-					(reference "C?")
+					(reference "C81")
 					(unit 1)
 				)
@@
 		(in_pos_files yes)
 		(dnp no)
-		(property "Reference" "C?"
+		(property "Reference" "C83"
 			(at 143.764 51.308 0)
 			(show_name no)
@@
 			(project "STM32-FPGA"
 				(path "/a5dcf55a-c00b-44e4-be21-50af8ba3dde4"
-					(reference "C?")
+					(reference "C83")
 					(unit 1)
 				)
@@
 		(in_pos_files yes)
 		(dnp no)
-		(property "Reference" "C?"
+		(property "Reference" "C87"
 			(at 179.324 51.308 0)
 			(show_name no)
@@
 			(project "STM32-FPGA"
 				(path "/a5dcf55a-c00b-44e4-be21-50af8ba3dde4"
-					(reference "C?")
+					(reference "C87")
 					(unit 1)
 				)
@@
 		(in_pos_files yes)
 		(dnp no)
-		(property "Reference" "C?"
+		(property "Reference" "C80"
 			(at 59.944 51.308 0)
 			(show_name no)
@@
 			(project "STM32-FPGA"
 				(path "/a5dcf55a-c00b-44e4-be21-50af8ba3dde4"
-					(reference "C?")
+					(reference "C80")
 					(unit 1)
 				)
@@
 		(in_pos_files yes)
 		(dnp no)
-		(property "Reference" "C?"
+		(property "Reference" "C86"
 			(at 170.434 51.308 0)
 			(show_name no)
@@
 			(project "STM32-FPGA"
 				(path "/a5dcf55a-c00b-44e4-be21-50af8ba3dde4"
-					(reference "C?")
+					(reference "C86")
 					(unit 1)
 				)
@@
 		(in_pos_files yes)
 		(dnp no)
-		(property "Reference" "C?"
+		(property "Reference" "C78"
 			(at 42.164 51.308 0)
 			(show_name no)
@@
 			(project "STM32-FPGA"
 				(path "/a5dcf55a-c00b-44e4-be21-50af8ba3dde4"
-					(reference "C?")
+					(reference "C78")
 					(unit 1)
 				)
@@
 	(sheet_instances
 		(path "/"
-			(page "11")
-		)
-	)
+			(page "6")
+		)
+	)
