File: stm32f103c8t6.kicad_sch (KiCad schematic)
At the start: 19 parts

Commit message: Hierarchy to Flat completes
The hierarchy sheets have been converted into flat sheets and global labels have been used in appropriate place.
Parts:
- added J?: Conn_01x04, symbol Connector_Generic:Conn_01x04
- gave numbers to parts that had none: 19
Connections:
- net +3V3: now also J?.4 (Pin_4)
- net GND: now also J?.1 (Pin_1)
- new net STM32_SWCLK_HED: J?.2 (Pin_2)
- new net STM32_SWDIO_HED: J?.3 (Pin_3)

Commit message: Decoupling done
The decoupling for the 10CL025 was completed using the evaluation module as reference.
Parts:
- gave numbers to parts that had none: 1
Changed lines of the file:
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@@
 		(in_pos_files yes)
 		(dnp yes)
-		(property "Reference" "J?"
+		(property "Reference" "J5"
 			(at 229.87 27.178 0)
 			(show_name no)
@@
 			(project "STM32-FPGA"
 				(path "/0d612cc7-7cb1-488a-a131-1e71117b8b3f"
-					(reference "J?")
+					(reference "J5")
 					(unit 1)
 				)
@@
 	(sheet_instances
 		(path "/"
-			(page "3")
+			(page "4")
 		)
 	)
