File: 10cl025yu256c8g.kicad_sch (KiCad schematic)
At the start: 24 parts

Commit message: No big changes made from last time
Other:
- note added: "All the power, decoupling and filtering connections are given as per the 10CL025 evaluation kit"
Changed lines of the file:
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@@
 	(generator_version "10.0")
 	(paper "A4")
+	(text "All the power, decoupling and filtering connections are given as per the 10CL025 evaluation kit\n"
+		(exclude_from_sim no)
+		(at 227.33 161.798 0)
+		(effects
+			(font
+				(size 1.27 1.27)
+			)
+		)
+	)
 	(junction
 		(at 39.37 153.67)
