File: 10cl025yu256c8g_io_bnks.kicad_sch (KiCad schematic)
At the start: 6 parts, among them Y4 ASE-50MHz

Commit message: No big changes made from last time
Connections:
- net PRFPGA_TCK: now also U5.H3 (TCK)
- net PRFPGA_TDI: now also U5.H4 (TDI)
- net PRFPGA_TDO: now also U5.J4 (TDO)
- net PRFPGA_TMS: now also U5.J5 (TMS)
- net FPGA_NSTATUS: now reaches U5.F4 (NSTATUS)
- net FPGA_NCOFIG: now reaches U5.H5 (NCONFIG)
- net FPGA_NCE: now reaches U5.J3 (NCE)
- net +3V3_FPGA renamed CL10_VCC_D_PLL
Changed lines of the file:
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@@
 	(wire
 		(pts
+			(xy 46.99 76.2) (xy 63.5 76.2)
+		)
+		(stroke
+			(width 0)
+			(type default)
+		)
+	)
+	(wire
+		(pts
 			(xy 85.09 217.17) (xy 85.09 223.52)
 		)
@@
 	(wire
 		(pts
+			(xy 46.99 68.58) (xy 63.5 68.58)
+		)
+		(stroke
+			(width 0)
+			(type default)
+		)
+	)
+	(wire
+		(pts
 			(xy 57.15 265.43) (xy 57.15 267.97)
 		)
@@
 	(wire
 		(pts
-			(xy 60.96 217.17) (xy 85.09 217.17)
+			(xy 46.99 73.66) (xy 63.5 73.66)
 		)
 		(stroke
@@
 	(wire
 		(pts
-			(xy 48.26 247.65) (xy 48.26 246.38)
+			(xy 60.96 217.17) (xy 85.09 217.17)
 		)
 		(stroke
@@
 	(wire
 		(pts
+			(xy 46.99 53.34) (xy 63.5 53.34)
+		)
+		(stroke
+			(width 0)
+			(type default)
+		)
+	)
+	(wire
+		(pts
 			(xy 78.74 228.6) (xy 85.09 228.6)
 		)
@@
 	(wire
 		(pts
+			(xy 46.99 71.12) (xy 63.5 71.12)
+		)
+		(stroke
+			(width 0)
+			(type default)
+		)
+	)
+	(wire
+		(pts
 			(xy 44.45 247.65) (xy 48.26 247.65)
 		)
@@
 	(wire
 		(pts
+			(xy 48.26 245.11) (xy 48.26 247.65)
+		)
+		(stroke
+			(width 0)
+			(type default)
+		)
+	)
+	(wire
+		(pts
 			(xy 44.45 248.92) (xy 44.45 247.65)
 		)
@@
 	(wire
 		(pts
+			(xy 46.99 78.74) (xy 63.5 78.74)
+		)
+		(stroke
+			(width 0)
+			(type default)
+		)
+	)
+	(wire
+		(pts
 			(xy 50.8 247.65) (xy 48.26 247.65)
 		)
@@
 	(wire
 		(pts
+			(xy 46.99 66.04) (xy 63.5 66.04)
+		)
+		(stroke
+			(width 0)
+			(type default)
+		)
+	)
+	(wire
+		(pts
 			(xy 44.45 256.54) (xy 44.45 261.62)
 		)
@@
 		)
 	)
+	(label "FPGA_JTAG_TDO"
+		(at 46.99 76.2 0)
+		(effects
+			(font
+				(size 1.27 1.27)
+			)
+			(justify left bottom)
+		)
+	)
+	(label "FPGA_NCE"
+		(at 46.99 78.74 0)
+		(effects
+			(font
+				(size 1.27 1.27)
+			)
+			(justify left bottom)
+		)
+	)
 	(label "FPGA_CLK_50MHz"
 		(at 43.18 228.6 0)
@@
 		)
 	)
+	(label "FPGA_NCOFIG"
+		(at 46.99 66.04 0)
+		(effects
+			(font
+				(size 1.27 1.27)
+			)
+			(justify left bottom)
+		)
+	)
 	(label "FPGA_JTAG_TDI"
 		(at 58.42 261.62 0)
@@
 	)
 	(label "FPGA_JTAG_TCK"
+		(at 46.99 71.12 0)
+		(effects
+			(font
+				(size 1.27 1.27)
+			)
+			(justify left bottom)
+		)
+	)
+	(label "FPGA_JTAG_TDI"
+		(at 46.99 68.58 0)
+		(effects
+			(font
+				(size 1.27 1.27)
+			)
+			(justify left bottom)
+		)
+	)
+	(label "FPGA_JTAG_TCK"
 		(at 58.42 265.43 0)
 		(effects
@@
 		)
 	)
+	(label "FPGA_JTAG_TMS"
+		(at 46.99 73.66 0)
+		(effects
+			(font
+				(size 1.27 1.27)
+			)
+			(justify left bottom)
+		)
+	)
+	(label "FPGA_NSTATUS"
+		(at 46.99 53.34 0)
+		(effects
+			(font
+				(size 1.27 1.27)
+			)
+			(justify left bottom)
+		)
+	)
 	(global_label "PRFPGA_TDO"
 		(shape bidirectional)
@@
 	)
 	(symbol
-		(lib_id "power:+3V3")
-		(at 48.26 246.38 0)
-		(unit 1)
-		(body_style 1)
-		(exclude_from_sim no)
-		(in_bom yes)
-		(on_board yes)
-		(in_pos_files yes)
-		(dnp no)
-		(property "Reference" "#PWR08"
-			(at 48.26 250.19 0)
-			(hide yes)
-			(show_name no)
-			(do_not_autoplace no)
-			(effects
-				(font
-					(size 1.27 1.27)
-				)
-			)
-		)
-		(property "Value" "+3V3_FPGA"
-			(at 48.26 242.316 0)
-			(show_name no)
-			(do_not_autoplace no)
-			(effects
-				(font
-					(size 1.27 1.27)
-				)
-			)
-		)
-		(property "Footprint" ""
-			(at 48.26 246.38 0)
-			(hide yes)
-			(show_name no)
-			(do_not_autoplace no)
-			(effects
-				(font
-					(size 1.27 1.27)
-				)
-			)
-		)
-		(property "Datasheet" ""
-			(at 48.26 246.38 0)
-			(hide yes)
-			(show_name no)
-			(do_not_autoplace no)
-			(effects
-				(font
-					(size 1.27 1.27)
-				)
-			)
-		)
-		(property "Description" "Power symbol creates a global label with name \"+3V3\""
-			(at 48.26 246.38 0)
-			(hide yes)
-			(show_name no)
-			(do_not_autoplace no)
-			(effects
-				(font
-					(size 1.27 1.27)
-				)
-			)
-		)
-		(pin "1"
-		)
-		(instances
-			(project "STM32-FPGA"
-				(path "/e1888878-1772-42cd-960b-88256a9714a3"
-					(reference "#PWR08")
-					(unit 1)
-				)
-			)
-		)
-	)
-	(symbol
 		(lib_id "power:GND")
 		(at 57.15 276.86 0)
@@
 				)
 			)
+		)
+	)
+	(symbol
+		(lib_id "power:VCC")
+		(at 48.26 245.11 0)
+		(unit 1)
+		(body_style 1)
+		(exclude_from_sim no)
+		(in_bom yes)
+		(on_board yes)
+		(in_pos_files yes)
+		(dnp no)
+		(property "Reference" "#PWR036"
+			(at 48.26 248.92 0)
+			(hide yes)
+			(show_name no)
+			(do_not_autoplace no)
+			(effects
+				(font
+					(size 1.27 1.27)
+				)
+			)
+		)
+		(property "Value" "CL10_VCC_D_PLL"
+			(at 40.132 241.046 0)
+			(show_name no)
+			(do_not_autoplace no)
+			(effects
+				(font
+					(size 1.27 1.27)
+				)
+				(justify left)
+			)
+		)
+		(property "Footprint" ""
+			(at 48.26 245.11 0)
+			(hide yes)
+			(show_name no)
+			(do_not_autoplace no)
+			(effects
+				(font
+					(size 1.27 1.27)
+				)
+			)
+		)
+		(property "Datasheet" ""
+			(at 48.26 245.11 0)
+			(hide yes)
+			(show_name no)
+			(do_not_autoplace no)
+			(effects
+				(font
+					(size 1.27 1.27)
+				)
+			)
+		)
+		(property "Description" "Power symbol creates a global label with name \"VCC\""
+			(at 48.26 245.11 0)
+			(hide yes)
+			(show_name no)
+			(do_not_autoplace no)
+			(effects
+				(font
+					(size 1.27 1.27)
+				)
+			)
+		)
+		(pin "1"
+		)
+		(instances
+			(project "STM32-FPGA"
+				(path "/e1888878-1772-42cd-960b-88256a9714a3"
+					(reference "#PWR036")
+					(unit 1)
+				)
+			)
