File: usb&power.kicad_sch (KiCad schematic)
At the start: 3 parts, among them J1 USB4105-GF-A-120

Commit message: No big changes made from last time
Other:
- note added: "Rajmohan thinks that power from 1 USB device itself will be sufficient enough if large current limiting resistors are added to it."
- moved on the sheet: J1, R8, R9
